Commit message: feat: independent gripper ros2_control, teach model, and dual-follower xacro
Split gripper hardware from the arm block, add piper_manipulation and teach
URDF entrypoints with meshes/tests, and drop host CAN bring-up from xacro.

Co-authored-by: Cursor <cursoragent@cursor.com>

File: urdf/parts/piper_arm.ros2_control.xacro (robot description, xacro)
@@ -2,5 +2,5 @@
 <robot xmlns:xacro="http://www.ros.org/wiki/xacro" name="piper_ros2_control">
   <xacro:macro name="piper_arm_ros2_control"
-    params="name:='PiperHardware' prefix:='' can_interface:='can0' init_can:='false' use_fake_hardware:='false' enable_gripper_control:='false' mit_kd_effort_damping:='0.0'">
+    params="name:='PiperHardware' prefix:='' can_interface:='can0' use_fake_hardware:='false' mit_kd_effort_damping:='0.0'">
     <ros2_control name="${name}" type="system">
       <hardware>
@@ -11,5 +11,4 @@
           <plugin>piper_hardware_interface/PiperHardwareInterface</plugin>
           <param name="can_interface">${can_interface}</param>
-          <param name="init_can">${init_can}</param>
           <!-- MIT effort-mode velocity damping. Default 0.0 keeps the ROS effort interface torque-transparent. -->
           <param name="mit_kd_effort_damping">${mit_kd_effort_damping}</param>
@@ -32,10 +31,4 @@
       <xacro:configure_joint joint_name="${prefix}joint5"/>
       <xacro:configure_joint joint_name="${prefix}joint6"/>
-      <xacro:if value="${enable_gripper_control}">
-        <joint name="${prefix}gripper_joint1">
-          <command_interface name="position"/>
-          <state_interface name="position"/>
-        </joint>
-      </xacro:if>
     </ros2_control>
   </xacro:macro>

File: urdf/piper.urdf.xacro (robot description, xacro)
@@ -6,5 +6,4 @@
   <xacro:arg name="rpy" default="0 0 0"/>
   <xacro:arg name="can_interface" default="can0"/>
-  <xacro:arg name="init_can" default="false"/>
   <xacro:arg name="ros2_control" default="true"/>
   <xacro:arg name="use_fake_hardware" default="false"/>
@@ -22,5 +21,4 @@
       prefix="$(arg prefix)"
       can_interface="$(arg can_interface)"
-      init_can="$(arg init_can)"
       use_fake_hardware="$(arg use_fake_hardware)"
       mit_kd_effort_damping="$(arg mit_kd_effort_damping)"/>

File: urdf/piper_with_gripper.urdf.xacro (robot description, xacro)
@@ -6,9 +6,9 @@
   <xacro:arg name="rpy" default="0 0 0"/>
   <xacro:arg name="can_interface" default="can0"/>
-  <xacro:arg name="init_can" default="false"/>
   <xacro:arg name="load_gripper" default="true"/>
   <xacro:arg name="ros2_control" default="true"/>
   <xacro:arg name="use_fake_hardware" default="false"/>
-  <xacro:arg name="enable_gripper_control" default="false"/>
+  <xacro:arg name="enable_gripper_control" default="true"/>
+  <xacro:arg name="gripper_home_on_activate" default="true"/>
   <xacro:arg name="mit_kd_effort_damping" default="0.0"/>
   <xacro:arg name="xyz_ee" default="0 0 0"/>
@@ -23,4 +23,5 @@
   <xacro:include filename="$(find piper_description)/urdf/parts/piper_gripper.xacro"/>
   <xacro:include filename="$(find piper_description)/urdf/parts/piper_arm.ros2_control.xacro"/>
+  <xacro:include filename="$(find piper_description)/urdf/parts/piper_gripper.ros2_control.xacro"/>
   <xacro:piper_arm
     prefix="$(arg prefix)"
@@ -43,8 +44,16 @@
       prefix="$(arg prefix)"
       can_interface="$(arg can_interface)"
-      init_can="$(arg init_can)"
       use_fake_hardware="$(arg use_fake_hardware)"
-      mit_kd_effort_damping="$(arg mit_kd_effort_damping)"
-      enable_gripper_control="$(arg enable_gripper_control)"/>
+      mit_kd_effort_damping="$(arg mit_kd_effort_damping)"/>
+    <xacro:if value="$(arg load_gripper)">
+      <xacro:if value="$(arg enable_gripper_control)">
+        <xacro:piper_gripper_ros2_control
+          name="PiperGripperHardware"
+          prefix="$(arg prefix)"
+          can_interface="$(arg can_interface)"
+          use_fake_hardware="$(arg use_fake_hardware)"
+          home_on_activate="$(arg gripper_home_on_activate)"/>
+      </xacro:if>
+    </xacro:if>
   </xacro:if>
 </robot>
