Commit message: feat: replace dual-arm xacro with experiment-table bimanual cell
Mount both Pipers on the table workbench, vendor table meshes, and treat gripper parent_link as absolute so prefixed flange links attach correctly.

Co-authored-by: Cursor <cursoragent@cursor.com>

File: urdf/parts/piper_gripper.xacro (robot description, xacro)
@@ -27,5 +27,7 @@
     <joint name="${prefix}gripper_base_joint" type="fixed">
       <origin xyz="${xyz_ee}" rpy="${rpy_ee}"/>
-      <parent link="${prefix}${parent_link}"/>
+      <!-- parent_link is absolute (do not apply prefix). Marvin uses flange_L;
+           Piper arms use left_flange_link / flange_link. -->
+      <parent link="${parent_link}"/>
       <child link="${prefix}gripper_base"/>
     </joint>

File: urdf/piper_bimanual_manipulation.urdf.xacro (robot description, xacro)
@@ -1,23 +1,25 @@
 <?xml version="1.0"?>
-<!-- Deployment-neutral left/right Piper composition. Values are injected by bringup. -->
-<robot xmlns:xacro="http://www.ros.org/wiki/xacro" name="piper_manipulation">
+<!-- Dual Piper + native grippers on the experiment table workbench.
+     Table meshes and arm mounts follow
+     https://github.com/Marco6-3/experiment_table_models
+     (left/right base at (±0.38, 0.32, 0.71), yaw=-90° toward the tabletop). -->
+<robot xmlns:xacro="http://www.ros.org/wiki/xacro" name="piper_bimanual_manipulation">
   <xacro:include filename="$(find piper_description)/urdf/parts/piper_arm.xacro"/>
   <xacro:include filename="$(find piper_description)/urdf/parts/piper_gripper.xacro"/>
   <xacro:include filename="$(find piper_description)/urdf/parts/piper_arm.ros2_control.xacro"/>
   <xacro:include filename="$(find piper_description)/urdf/parts/piper_gripper.ros2_control.xacro"/>
+  <xacro:include filename="$(find piper_description)/urdf/parts/experiment_table.xacro"/>
   <xacro:include filename="$(find pika_gripper_description)/urdf/pika_gripper.xacro"/>
   <xacro:include filename="$(find pika_gripper_description)/urdf/pika_gripper.ros2_control.xacro"/>
   <xacro:arg name="enable_left" default="true"/>
   <xacro:arg name="enable_right" default="true"/>
+  <xacro:arg name="enable_table" default="true"/>
   <xacro:arg name="use_fake_hardware" default="true"/>
   <xacro:arg name="left_can_interface" default="can0"/>
   <xacro:arg name="right_can_interface" default="can1"/>
-  <!-- End-effector selection is per side: at most one of the two flags below
-       may be true for a given side. The controller_bringup launch file
-       derives both flags from one validated `<side>_end_effector` argument
-       (none | piper_gripper | pika_gripper) so unsupported values fail
-       launch instead of silently producing a partial robot model. -->
-  <xacro:arg name="enable_left_gripper" default="false"/>
-  <xacro:arg name="enable_right_gripper" default="false"/>
+  <!-- Default: Piper gripper per side. Bringup maps
+       <side>_end_effector (none | piper_gripper | pika_gripper) onto these. -->
+  <xacro:arg name="enable_left_gripper" default="true"/>
+  <xacro:arg name="enable_right_gripper" default="true"/>
   <xacro:arg name="left_gripper_home_on_activate" default="true"/>
   <xacro:arg name="right_gripper_home_on_activate" default="true"/>
@@ -26,12 +28,15 @@
   <xacro:arg name="left_gripper_serial_port" default="/dev/ttyUSB0"/>
   <xacro:arg name="right_gripper_serial_port" default="/dev/ttyUSB1"/>
-  <xacro:arg name="left_xyz" default="0 0.30 0"/>
-  <xacro:arg name="right_xyz" default="0 -0.30 0"/>
-  <xacro:arg name="left_rpy" default="0 0 0"/>
-  <xacro:arg name="right_rpy" default="0 0 0"/>
+  <xacro:arg name="left_xyz" default="-0.38 0.32 0.71"/>
+  <xacro:arg name="right_xyz" default="0.38 0.32 0.71"/>
+  <xacro:arg name="left_rpy" default="0 0 -1.57079632679"/>
+  <xacro:arg name="right_rpy" default="0 0 -1.57079632679"/>
   <xacro:property
     name="gripper_tcp"
     value="${xacro.load_yaml('$(find piper_description)/config/gripper_tcp.yaml')}"/>
   <link name="world"/>
+  <xacro:if value="$(arg enable_table)">
+    <xacro:experiment_table prefix="table_" parent="world" xyz="0 0 0" rpy="0 0 0"/>
+  </xacro:if>
   <xacro:if value="$(arg enable_left)">
     <joint name="world_to_left_mount" type="fixed">
@@ -41,5 +46,5 @@
     <xacro:piper_arm prefix="left_" connected_to="left_mount"/>
     <xacro:piper_arm_ros2_control
-      name="LeftPiperHardware" prefix="left_"
+      name="left_piper_hardware" prefix="left_"
       can_interface="$(arg left_can_interface)"
       use_fake_hardware="$(arg use_fake_hardware)"/>
@@ -47,9 +52,9 @@
       <xacro:piper_gripper
         prefix="left_"
-        parent_link="flange_link"
+        parent_link="left_flange_link"
         tcp_xyz="${gripper_tcp['origin']['xyz']}"
         tcp_rpy="${gripper_tcp['origin']['rpy']}"/>
       <xacro:piper_gripper_ros2_control
-        name="LeftPiperGripperHardware" prefix="left_"
+        name="left_piper_gripper_hardware" prefix="left_"
         can_interface="$(arg left_can_interface)"
         use_fake_hardware="$(arg use_fake_hardware)"
@@ -73,5 +78,5 @@
     <xacro:piper_arm prefix="right_" connected_to="right_mount"/>
     <xacro:piper_arm_ros2_control
-      name="RightPiperHardware" prefix="right_"
+      name="right_piper_hardware" prefix="right_"
       can_interface="$(arg right_can_interface)"
       use_fake_hardware="$(arg use_fake_hardware)"/>
@@ -79,9 +84,9 @@
       <xacro:piper_gripper
         prefix="right_"
-        parent_link="flange_link"
+        parent_link="right_flange_link"
         tcp_xyz="${gripper_tcp['origin']['xyz']}"
         tcp_rpy="${gripper_tcp['origin']['rpy']}"/>
       <xacro:piper_gripper_ros2_control
-        name="RightPiperGripperHardware" prefix="right_"
+        name="right_piper_gripper_hardware" prefix="right_"
         can_interface="$(arg right_can_interface)"
         use_fake_hardware="$(arg use_fake_hardware)"

File: urdf/piper_with_gripper.urdf.xacro (robot description, xacro)
@@ -33,5 +33,5 @@
     <xacro:piper_gripper
       prefix="$(arg prefix)"
-      parent_link="flange_link"
+      parent_link="$(arg prefix)flange_link"
       xyz_ee="$(arg xyz_ee)"
       rpy_ee="$(arg rpy_ee)"
