Commit message: feat: keep bimanual mounts in xacro and add visual mounting plates
Visualize launches no longer hardcode arm poses, so site-calibrated xyz and
the 260x100x10 mm plates take effect without a second source of truth.

Co-authored-by: Cursor <cursoragent@cursor.com>

File: urdf/piper_bimanual_manipulation.urdf.xacro (robot description, xacro)
@@ -3,5 +3,6 @@
      Table meshes and arm mounts follow
      https://github.com/Marco6-3/experiment_table_models
-     (left/right base at (±0.38, 0.32, 0.71), yaw=-90° toward the tabletop). -->
+     (site-calibrated left_xyz / right_xyz; CAD reference was
+     ±0.38, 0.32, 0.71, yaw=-90° toward the tabletop). -->
 <robot xmlns:xacro="http://www.ros.org/wiki/xacro" name="piper_bimanual_manipulation">
   <xacro:include filename="$(find piper_description)/urdf/parts/piper_arm.xacro"/>
@@ -10,9 +11,16 @@
   <xacro:include filename="$(find piper_description)/urdf/parts/piper_gripper.ros2_control.xacro"/>
   <xacro:include filename="$(find piper_description)/urdf/parts/experiment_table.xacro"/>
+  <xacro:include filename="$(find piper_description)/urdf/parts/piper_mounting_plate.xacro"/>
   <xacro:arg name="enable_left" default="true"/>
   <xacro:arg name="enable_right" default="true"/>
+  <xacro:arg name="connected_to" default="world"/>
+  <xacro:arg name="enable_table" default="true"/>
+  <xacro:arg name="table_xyz" default="0 0 0"/>
+  <xacro:arg name="table_rpy" default="0 0 0"/>
   <xacro:arg name="use_fake_hardware" default="true"/>
   <xacro:arg name="left_can_interface" default="can0"/>
   <xacro:arg name="right_can_interface" default="can1"/>
+  <xacro:arg name="left_mit_kd_effort_damping" default="0.0"/>
+  <xacro:arg name="right_mit_kd_effort_damping" default="0.0"/>
   <!-- Default: Piper gripper per side. Bringup maps
        <side>_end_effector (none | piper_gripper | pika_gripper) onto these. -->
@@ -25,6 +33,6 @@
   <xacro:arg name="left_gripper_serial_port" default="/dev/ttyUSB0"/>
   <xacro:arg name="right_gripper_serial_port" default="/dev/ttyUSB1"/>
-  <xacro:arg name="left_xyz" default="-0.38 0.32 0.71"/>
-  <xacro:arg name="right_xyz" default="0.38 0.32 0.71"/>
+  <xacro:arg name="left_xyz" default="-0.32 0.29 0.72"/>
+  <xacro:arg name="right_xyz" default="0.32 0.29 0.72"/>
   <xacro:arg name="left_rpy" default="0 0 -1.57079632679"/>
   <xacro:arg name="right_rpy" default="0 0 -1.57079632679"/>
@@ -44,17 +52,28 @@
     name="gripper_tcp"
     value="${xacro.load_yaml('$(find piper_description)/config/gripper_tcp.yaml')}"/>
-  <link name="world"/>
+  <link name="$(arg connected_to)"/>
   <!-- Visual-only; no <collision>. Planner world cuboids own table collision. -->
-  <xacro:experiment_table prefix="table_" parent="world" xyz="0 0 0" rpy="0 0 0"/>
+  <xacro:if value="$(arg enable_table)">
+    <xacro:experiment_table
+      prefix="table_"
+      parent="$(arg connected_to)"
+      xyz="$(arg table_xyz)"
+      rpy="$(arg table_rpy)"/>
+  </xacro:if>
   <xacro:if value="$(arg enable_left)">
     <joint name="world_to_left_mount" type="fixed">
-      <parent link="world"/><child link="left_mount"/>
+      <parent link="$(arg connected_to)"/><child link="left_mount"/>
       <origin xyz="$(arg left_xyz)" rpy="$(arg left_rpy)"/>
     </joint>
+    <xacro:piper_mounting_plate
+      prefix="left_"
+      parent="$(arg connected_to)"
+      xyz="$(arg left_xyz)"/>
     <xacro:piper_arm prefix="left_" connected_to="left_mount"/>
     <xacro:piper_arm_ros2_control
       name="left_piper_hardware" prefix="left_"
       can_interface="$(arg left_can_interface)"
-      use_fake_hardware="$(arg use_fake_hardware)"/>
+      use_fake_hardware="$(arg use_fake_hardware)"
+      mit_kd_effort_damping="$(arg left_mit_kd_effort_damping)"/>
     <xacro:if value="$(arg enable_left_gripper)">
       <xacro:piper_gripper
@@ -81,12 +100,17 @@
   <xacro:if value="$(arg enable_right)">
     <joint name="world_to_right_mount" type="fixed">
-      <parent link="world"/><child link="right_mount"/>
+      <parent link="$(arg connected_to)"/><child link="right_mount"/>
       <origin xyz="$(arg right_xyz)" rpy="$(arg right_rpy)"/>
     </joint>
+    <xacro:piper_mounting_plate
+      prefix="right_"
+      parent="$(arg connected_to)"
+      xyz="$(arg right_xyz)"/>
     <xacro:piper_arm prefix="right_" connected_to="right_mount"/>
     <xacro:piper_arm_ros2_control
       name="right_piper_hardware" prefix="right_"
       can_interface="$(arg right_can_interface)"
-      use_fake_hardware="$(arg use_fake_hardware)"/>
+      use_fake_hardware="$(arg use_fake_hardware)"
+      mit_kd_effort_damping="$(arg right_mit_kd_effort_damping)"/>
     <xacro:if value="$(arg enable_right_gripper)">
       <xacro:piper_gripper
